File: schematics/ICPSLC24-10NA.kicad_sch (KiCad schematic)
At the start: 35 parts, among them J1 Debug, K1 Reset, M1 TRÅDFRI, Q1 FDD880; 30V, 58A, 9mΩ

Commit message: update
Parts:
- D3: footprint (none) -> RS1M:SMA_DIO
- K1: footprint (none) -> PTS641SM34SMTR2LFS:PTS641
- M1: footprint (none) -> icc-1:ICC-1_POLY_PCB2.0
- Q1: footprint TO_SOT_Packages_SMD:TO-252-2_Rectifier -> FDD8880:DPAK_ONS
- R10, R2, R4, R5, R9: footprint (none) -> Resistor_SMD:R_0805_2012Metric_Pad1.20x1.40mm_HandSolder
Changed lines of the file:
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@@
     (effects (font (size 1.524 1.524)) (justify left bottom))
   )
-  (label "SW1" (at 88.9 78.74 0)
+  (label "SW1" (at 88.9 78.74 0) (fields_autoplaced)
     (effects (font (size 1.524 1.524)) (justify left bottom))
   )
-  (label "SWCLK" (at 40.64 34.29 180)
-    (effects (font (size 1.524 1.524)) (justify right bottom))
-  )
-  (label "OUT_SENSE" (at 88.9 81.28 0)
+  (label "SWCLK" (at 40.64 34.29 180) (fields_autoplaced)
+    (effects (font (size 1.524 1.524)) (justify right bottom))
+  )
+  (label "OUT_SENSE" (at 88.9 81.28 0) (fields_autoplaced)
     (effects (font (size 1.524 1.524)) (justify left bottom))
   )
-  (label "SWDIO" (at 40.64 36.83 180)
-    (effects (font (size 1.524 1.524)) (justify right bottom))
-  )
-  (label "SW1" (at 69.85 86.36 180)
-    (effects (font (size 1.524 1.524)) (justify right bottom))
-  )
-  (label "SWDIO" (at 137.16 83.82 180)
-    (effects (font (size 1.524 1.524)) (justify right bottom))
-  )
-  (label "PWM1" (at 151.13 91.44 0)
+  (label "SWDIO" (at 40.64 36.83 180) (fields_autoplaced)
+    (effects (font (size 1.524 1.524)) (justify right bottom))
+  )
+  (label "SW1" (at 69.85 86.36 180) (fields_autoplaced)
+    (effects (font (size 1.524 1.524)) (justify right bottom))
+  )
+  (label "SWDIO" (at 137.16 83.82 180) (fields_autoplaced)
+    (effects (font (size 1.524 1.524)) (justify right bottom))
+  )
+  (label "PWM1" (at 151.13 91.44 0) (fields_autoplaced)
     (effects (font (size 1.524 1.524)) (justify left bottom))
   )
-  (label "SWCLK" (at 137.16 81.28 180)
-    (effects (font (size 1.524 1.524)) (justify right bottom))
-  )
-  (label "PWM1" (at 88.9 86.36 0)
+  (label "SWCLK" (at 137.16 81.28 180) (fields_autoplaced)
+    (effects (font (size 1.524 1.524)) (justify right bottom))
+  )
+  (label "PWM1" (at 88.9 86.36 0) (fields_autoplaced)
     (effects (font (size 1.524 1.524)) (justify left bottom))
   )
-  (label "OUT_SENSE" (at 252.73 93.98 180)
+  (label "OUT_SENSE" (at 252.73 93.98 180) (fields_autoplaced)
     (effects (font (size 1.524 1.524)) (justify right bottom))
   )
@@
       (effects (font (size 1.27 1.27)) (justify left))
     )
-    (property "Footprint" "TO_SOT_Packages_SMD:TO-252-2_Rectifier" (at 181.61 88.9 0)
+    (property "Footprint" "FDD8880:DPAK_ONS" (at 181.61 88.9 0)
       (effects (font (size 1.27 1.27)) hide)
     )
@@
       (effects (font (size 1.524 1.524)))
     )
-    (property "Footprint" "" (at 120.65 78.74 0)
-      (effects (font (size 1.524 1.524)) hide)
+    (property "Footprint" "icc-1:ICC-1_POLY_PCB2.0" (at 120.65 78.74 0)
+      (effects (font (size 1.524 1.524)))
     )
     (property "Datasheet" "" (at 120.65 78.74 0)
@@
       (effects (font (size 1.27 1.27)))
     )
-    (property "Footprint" "" (at 179.07 78.74 0)
+    (property "Footprint" "RS1M:SMA_DIO" (at 179.07 78.74 0)
       (effects (font (size 1.27 1.27)) hide)
     )
@@
       (effects (font (size 1.27 1.27)))
     )
-    (property "Footprint" "" (at 57.15 95.25 0)
+    (property "Footprint" "PTS641SM34SMTR2LFS:PTS641" (at 57.15 95.25 0)
       (effects (font (size 1.27 1.27)) hide)
     )
@@
       (effects (font (size 1.27 1.27)))
     )
-    (property "Footprint" "" (at 60.452 78.74 90)
+    (property "Footprint" "Resistor_SMD:R_0805_2012Metric_Pad1.20x1.40mm_HandSolder" (at 60.452 78.74 90)
       (effects (font (size 1.27 1.27)) hide)
     )
@@
       (effects (font (size 1.27 1.27)))
     )
-    (property "Footprint" "" (at 162.56 89.662 90)
+    (property "Footprint" "Resistor_SMD:R_0805_2012Metric_Pad1.20x1.40mm_HandSolder" (at 162.56 89.662 90)
       (effects (font (size 1.27 1.27)) hide)
     )
@@
       (effects (font (size 1.27 1.27)))
     )
-    (property "Footprint" "" (at 167.132 96.52 90)
+    (property "Footprint" "Resistor_SMD:R_0805_2012Metric_Pad1.20x1.40mm_HandSolder" (at 167.132 96.52 90)
       (effects (font (size 1.27 1.27)) hide)
     )
@@
       (effects (font (size 1.27 1.27)))
     )
-    (property "Footprint" "" (at 220.472 87.63 90)
+    (property "Footprint" "Resistor_SMD:R_0805_2012Metric_Pad1.20x1.40mm_HandSolder" (at 220.472 87.63 90)
       (effects (font (size 1.27 1.27)) hide)
     )
@@
       (effects (font (size 1.27 1.27)))
     )
-    (property "Footprint" "" (at 220.472 100.33 90)
-      (effects (font (size 1.27 1.27)) hide)
-    )
+    (property "Footprint" "Resistor_SMD:R_0805_2012Metric_Pad1.20x1.40mm_HandSolder" (at 220.472 100.33 90)
+      (effects (font (size 1.27 1.27)) hide)
+    )
